File: ardIOExp.brd (EAGLE design)
At the start: 89.6 x 50 mm, 45 parts, among them CON1 GND 12V, U1 L78D2TT

Commit message: change name of voltage regulator
Parts:
- renumbered U1 to V_REG_5V
Changed lines of the file:
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@@
 <element name="U$6" library="ALX_LIB" package="HALX2_532_SILKSCREEN" value="" x="86.995" y="34.163" rot="R90"/>
 <element name="U$7" library="ALX_LIB" package="HALX2_532_TSTOP" value="" x="5.588" y="35.814"/>
-<element name="U1" library="L78" package="D2PAK" value="L78D2TT" x="15.367" y="7.366" rot="R180"/>
+<element name="V_REG_5V" library="L78" package="D2PAK" value="L78D2TT" x="15.367" y="7.366" rot="R180"/>
 </elements>
 <signals>
@@
 <wire x1="10.16" y1="29.845" x2="10.16" y2="27.305" width="0.6096" layer="16"/>
 <wire x1="5.08" y1="45.085" x2="5.08" y2="47.625" width="0.6096" layer="16"/>
-<contactref element="U1" pad="2"/>
+<contactref element="V_REG_5V" pad="2"/>
 <polygon width="0.4064" layer="1" isolate="0.4064" rank="3">
 <vertex x="0" y="2.54"/>
@@
 <contactref element="SV3" pad="5"/>
 <contactref element="C9" pad="1"/>
-<contactref element="U1" pad="1"/>
+<contactref element="V_REG_5V" pad="1"/>
 <wire x1="17.907" y1="19.177" x2="17.907" y2="15.621" width="1.27" layer="1"/>
 <wire x1="17.907" y1="19.177" x2="16.383" y2="20.701" width="1.27" layer="16"/>
@@
 <wire x1="74.041" y1="28.067" x2="71.755" y2="28.067" width="0.6096" layer="1"/>
 <wire x1="71.755" y1="28.067" x2="71.755" y2="28.155" width="0.8128" layer="1"/>
-<contactref element="U1" pad="3"/>
+<contactref element="V_REG_5V" pad="3"/>
 <via x="12.827" y="22.479" extent="1-16" drill="0.9" shape="octagon"/>
 <via x="14.478" y="22.479" extent="1-16" drill="0.9" shape="octagon"/>
